Commit message: TurtleBot3 mobile manipulation: fetch and deliver with Nav2, MoveIt 2 and py_trees

File: fetch_deliver_description/urdf/gazebo/turtlebot3_waffle_pi.gazebo.xacro (robot description, xacro)
@@ -6,6 +6,6 @@
 <robot xmlns:xacro="http://ros.org/wiki/xacro">
   <xacro:macro name="turtlebot3_waffle_pi_gazebo" params="prefix">
-  <xacro:property name="laser_visual"  value="true"/>
-  <xacro:property name="camera_visual" value="true"/>
+  <xacro:property name="laser_visual"  value="false"/>
+  <xacro:property name="camera_visual" value="false"/>
   <xacro:property name="imu_visual"    value="true"/>
   <gazebo reference="${prefix}base_link">
